Commit message: wheels possition change

File: description/robot_core.xacro (robot description, xacro)
@@ -25,5 +25,5 @@
         <parent link="base_link"/>
         <child link="chassis"/>
-        <origin xyz="-0.1 0.0 0.0"/>
+        <origin xyz="-0.15 0.0 0.0"/>
     </joint>
     <link name="chassis">
@@ -91,11 +91,77 @@
         </xacro:inertial_cylinder>
     </link>
-    <!-- Caster Wheel -->
-    <joint name="caster_wheel_joint" type="fixed">
+    <!-- Caster Wheel 1-->
+    <joint name="caster_wheel_1_joint" type="fixed">
         <parent link="chassis"/>
-        <child link="caster_wheel"/>
-        <origin xyz="0.24 0.0 0.0"/>
+        <child link="caster_wheel_1"/>
+        <origin xyz="0.24 0.1 0.0"/>
     </joint>
-    <link name="caster_wheel">
+    <link name="caster_wheel_1">
+        <visual>
+            <geometry>
+                <sphere radius="0.05"/>
+            </geometry>
+            <material name="white"/>
+        </visual>
+        <collision>
+            <geometry>
+                <sphere radius="0.05"/>
+            </geometry>
+        </collision>
+        <xacro:inertial_sphere mass="0.1" radius="0.05">
+             <origin xyz="0 0 0" rpy="0.0 0.0 0.0"/>
+        </xacro:inertial_sphere>
+    </link>
+     <!-- Caster Wheel 2-->
+    <joint name="caster_wheel_2_joint" type="fixed">
+        <parent link="chassis"/>
+        <child link="caster_wheel_2"/>
+        <origin xyz="0.06 0.1 0.0"/>
+    </joint>
+    <link name="caster_wheel_2">
+        <visual>
+            <geometry>
+                <sphere radius="0.05"/>
+            </geometry>
+            <material name="white"/>
+        </visual>
+        <collision>
+            <geometry>
+                <sphere radius="0.05"/>
+            </geometry>
+        </collision>
+        <xacro:inertial_sphere mass="0.1" radius="0.05">
+             <origin xyz="0 0 0" rpy="0.0 0.0 0.0"/>
+        </xacro:inertial_sphere>
+    </link>
+    <!-- Caster Wheel 3-->
+    <joint name="caster_wheel_3_joint" type="fixed">
+        <parent link="chassis"/>
+        <child link="caster_wheel_3"/>
+        <origin xyz="0.06 -0.1 0.0"/>
+    </joint>
+    <link name="caster_wheel_3">
+        <visual>
+            <geometry>
+                <sphere radius="0.05"/>
+            </geometry>
+            <material name="white"/>
+        </visual>
+        <collision>
+            <geometry>
+                <sphere radius="0.05"/>
+            </geometry>
+        </collision>
+        <xacro:inertial_sphere mass="0.1" radius="0.05">
+             <origin xyz="0 0 0" rpy="0.0 0.0 0.0"/>
+        </xacro:inertial_sphere>
+    </link>
+    <!-- Caster Wheel 4-->
+    <joint name="caster_wheel_4_joint" type="fixed">
+        <parent link="chassis"/>
+        <child link="caster_wheel_4"/>
+        <origin xyz="0.24 -0.1 0.0"/>
+    </joint>
+    <link name="caster_wheel_4">
         <visual>
             <geometry>

Commit message: gazebo sim spawn working, teleop plugin not working

File: description/robot_core.xacro (robot description, xacro)
@@ -45,4 +45,7 @@
         </xacro:inertial_box>
     </link>
+    <gazebo reference="chassis">
+        <material> Gazebo/Purple</material>
+    </gazebo>
     <!-- Left Wheel -->
     <joint name="left_wheel_joint" type="continuous">
@@ -68,4 +71,7 @@
         </xacro:inertial_cylinder>
     </link>
+    <gazebo reference="left_wheel">
+        <material> Gazebo/Black</material>
+    </gazebo>
     <!-- Rigth Wheel -->
     <joint name="right_wheel_joint" type="continuous">
@@ -91,4 +97,7 @@
         </xacro:inertial_cylinder>
     </link>
+    <gazebo reference="right_wheel">
+        <material> Gazebo/Black</material>
+    </gazebo>
     <!-- Caster Wheel 1-->
     <joint name="caster_wheel_1_joint" type="fixed">
@@ -109,8 +118,11 @@
             </geometry>
         </collision>
-        <xacro:inertial_sphere mass="0.1" radius="0.05">
-             <origin xyz="0 0 0" rpy="0.0 0.0 0.0"/>
-        </xacro:inertial_sphere>
-    </link>
+        <xacro:inertial_sphere mass="0.01" radius="0.05">
+             <origin xyz="0 0 0" rpy="0.0 0.0 0.0"/>
+        </xacro:inertial_sphere>
+    </link>
+    <gazebo reference="caster_wheel_1">
+        <material> Gazebo/White</material>
+    </gazebo>
      <!-- Caster Wheel 2-->
     <joint name="caster_wheel_2_joint" type="fixed">
@@ -131,8 +143,11 @@
             </geometry>
         </collision>
-        <xacro:inertial_sphere mass="0.1" radius="0.05">
-             <origin xyz="0 0 0" rpy="0.0 0.0 0.0"/>
-        </xacro:inertial_sphere>
-    </link>
+        <xacro:inertial_sphere mass="0.01" radius="0.05">
+             <origin xyz="0 0 0" rpy="0.0 0.0 0.0"/>
+        </xacro:inertial_sphere>
+    </link>
+    <gazebo reference="caster_wheel_2">
+        <material> Gazebo/White</material>
+    </gazebo>
     <!-- Caster Wheel 3-->
     <joint name="caster_wheel_3_joint" type="fixed">
@@ -153,8 +168,11 @@
             </geometry>
         </collision>
-        <xacro:inertial_sphere mass="0.1" radius="0.05">
-             <origin xyz="0 0 0" rpy="0.0 0.0 0.0"/>
-        </xacro:inertial_sphere>
-    </link>
+        <xacro:inertial_sphere mass="0.01" radius="0.05">
+             <origin xyz="0 0 0" rpy="0.0 0.0 0.0"/>
+        </xacro:inertial_sphere>
+    </link>
+    <gazebo reference="caster_wheel_3">
+        <material> Gazebo/White</material>
+    </gazebo>
     <!-- Caster Wheel 4-->
     <joint name="caster_wheel_4_joint" type="fixed">
@@ -175,7 +193,10 @@
             </geometry>
         </collision>
-        <xacro:inertial_sphere mass="0.1" radius="0.05">
-             <origin xyz="0 0 0" rpy="0.0 0.0 0.0"/>
-        </xacro:inertial_sphere>
-    </link>
+        <xacro:inertial_sphere mass="0.01" radius="0.05">
+             <origin xyz="0 0 0" rpy="0.0 0.0 0.0"/>
+        </xacro:inertial_sphere>
+    </link>
+    <gazebo reference="caster_wheel_4">
+        <material> Gazebo/White</material>
+    </gazebo>
 </robot>
